File: pcb/pcb/pcb.kicad_pcb (KiCad board)
At the start: 2 copper layers, 8 parts, among them J1 Connection 1, J2 Connection 2, J3 Motor1, J4 Motor2, J5 Motor4, J6 Motor3, J7 Bateria, J8 Motor3

Commit message: Update pcb
Parts:
- moved J7 0.90 mm to (144.1, 112.5), turned to 90 degrees
Routing:
- net Net-(J1-Pin_1): track 0.00 -> 81.0 mm
- net Net-(J1-Pin_2): track 0.00 -> 52.9 mm
